File: hardware/wo_poe/ethernet-extension.kicad_pcb (KiCad board)
At the start: 2 copper layers, 40 x 40 mm, 60 parts, among them J1 STACK-UP-HIGH, J2 STACK-DOWN, J3 STACK-UP-HIGH, J4 STACK-DOWN, P1 RJPSL-001TA1, U1 W5500, U2 M24C64, U3 DRILL, U4 DRILL, U5 DRILL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

Commit message: Add 3d information (final)
Parts:
- C10, C11, C12, C15, C16, C17, C2, C20, C3, C5, C6, C7, C8, L1, L2: footprint kicad-libraries:0603 -> kicad-libraries:C0603
- C18, C19, C9: footprint kicad-libraries:0805 -> kicad-libraries:C0805
- C21: footprint kicad-libraries:1206 -> kicad-libraries:C1206
- G***: footprint Logo_31x31 -> kicad-libraries:Logo_31x31
- R1, R10, R11, R12, R13, R14, R2, R3, R4, R5, R6, R7, R8, R9: footprint kicad-libraries:0603 -> kicad-libraries:R0603
- VAL: footprint WEEE_7mm -> kicad-libraries:WEEE_7mm
- VAL: footprint CE_5mm -> kicad-libraries:CE_5mm
- turned VAL to 180 degrees
Connections:
- FILTER1 pad 13: (no net) -> Net-(FILTER1-Pad13)
- FILTER1 pad 14: (no net) -> Net-(FILTER1-Pad14)
- FILTER1 pad 3: (no net) -> Net-(FILTER1-Pad3)
- FILTER1 pad 4: (no net) -> Net-(FILTER1-Pad4)
- J1 pad 25: (no net) -> Net-(J1-Pad25)
- J1 pad 27: (no net) -> Net-(J1-Pad27)
- J1 pad 29: (no net) -> Net-(J1-Pad29)
- J2 pad 23: (no net) -> Net-(J2-Pad23)
- P1 pad 10: (no net) -> Net-(P1-Pad10)
- P1 pad 11: (no net) -> Net-(P1-Pad11)
- P1 pad 12: (no net) -> Net-(P1-Pad12)
- P1 pad 9: (no net) -> Net-(P1-Pad9)
- U1 pad 12: (no net) -> Net-(U1-Pad12)
- U1 pad 13: (no net) -> Net-(U1-Pad13)
- U1 pad 18: (no net) -> Net-(U1-Pad18)
- U1 pad 24: (no net) -> Net-(U1-Pad24)
- U1 pad 26: (no net) -> Net-(U1-Pad26)
- U1 pad 27: (no net) -> Net-(U1-Pad27)
- U1 pad 46: (no net) -> Net-(U1-Pad46)
- U1 pad 47: (no net) -> Net-(U1-Pad47)
- U1 pad 7: (no net) -> Net-(U1-Pad7)
- U2 pad 7: (no net) -> Net-(U2-Pad7)
