File: hardware/wo_poe/ethernet-extension-wopoe.kicad_pcb (KiCad board)
At the start: 2 copper layers, 40 x 40 mm, 60 parts, among them J1 STACK-UP-HIGH, J2 STACK-DOWN, J3 STACK-UP-HIGH, J4 STACK-DOWN, P1 RJPSL-001TA1, U1 W5500, U2 M24C64, U3 DRILL, U4 DRILL, U5 DRILL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

Commit message: add data of ethernet extension 1.1
move to kicad 6
Parts:
- removed FILTER1: IP4254CZ16-8, kicad-libraries:DFN16-33x135
- removed R4: 10k, kicad-libraries:R0603
- removed RP1: 10k, kicad-libraries:4X0603
- added C101: 10pF, kicad-libraries:C0402F, B.Cu at (162.4, 121.7)
- added C102: 4.7uF, kicad-libraries:C0805, B.Cu at (140.3, 115.3)
- added C103: 4.7uF, kicad-libraries:C0805, B.Cu at (137.9, 121.7)
- added D101: ‎PESD3V3L1BA, kicad-libraries:SOD-323, B.Cu at (145.4, 100.5)
- added L101: TBD, kicad-libraries:R0603F, B.Cu at (133.6, 119.4)
- added R101: 33, kicad-libraries:R0402F, F.Cu at (152.5, 108.5)
- added R102: 33, kicad-libraries:R0402F, F.Cu at (153.2, 107.8)
- added R103: 33, kicad-libraries:R0402F, F.Cu at (150.9, 110.0)
- added R104: 33, kicad-libraries:R0402F, F.Cu at (151.6, 109.3)
- added R105: 1k, kicad-libraries:R0603, F.Cu at (161.6, 116.2)
- added R106: DNP, kicad-libraries:R0603, F.Cu at (161.6, 117.7)
- added RP102: 82, kicad-libraries:4X0402, B.Cu at (161.3, 123.8)
- added RP103: DNP, kicad-libraries:4X0402, F.Cu at (161.3, 123.8)
- added U101: AZ1117-3V3, kicad-libraries:SOT-223, B.Cu at (143.2, 121.0)
- R10, R11: value 82 -> 49.9
- R2: value 10k -> DNP
- moved R1 6.25 mm to (158.7, 116.2), turned to 180 degrees
- moved R2 6.16 mm to (158.7, 117.7), turned to 180 degrees
- moved C4 1.11 mm to (144.5, 111.3), turned to 90 degrees
Connections:
- net Net-(C21-Pad1) renamed SHD
- net Net-(J3-Pad22) renamed S5V
- C18 pad 1: RXIP -> Net-(C18-Pad1)
- C19 pad 1: RXIN -> Net-(C19-Pad1)
- C20 pad 2: 3V3 -> VCC
- J3 pad 28: VCC -> S3V3
- J4 pad 28: VCC -> S3V3
- P1 pad 1: TXOP -> Net-(P1-Pad1)
- P1 pad 14: +3.3VP -> 3V3
- P1 pad 2: TXON -> Net-(P1-Pad2)
- P1 pad 8: +3.3VP -> 3V3
- R10 pad 1: RXIP -> Net-(C18-Pad1)
- R11 pad 2: RXIN -> Net-(C19-Pad1)
- R7 pad 2: TXOP -> Net-(P1-Pad1)
- R8 pad 2: TXON -> Net-(P1-Pad2)
- U2 pad 8: 3V3 -> VCC
Routing:
- net VCC: track 15.0 -> 74.0 mm, vias 1 -> 3
- net GND: track 347.8 -> 320.8 mm, vias 80 -> 128
- net 3V3: track 57.7 -> 83.7 mm
- net +3.3VP: track 75.2 -> 55.8 mm, vias 8 -> 6
- net TXON: track 19.5 -> 3.82 mm, vias 1 -> 0
- net Net-(P1-Pad2): track 0.00 -> 15.2 mm, vias 0 -> 1
- net Net-(P1-Pad1): track 0.00 -> 14.8 mm, vias 0 -> 1
- net TXOP: track 18.0 -> 3.71 mm, vias 1 -> 0
- net S5V: track 11.0 -> 21.4 mm
- net SHD: track 5.14 -> 13.6 mm, vias 0 -> 7
- net S3V3: track 0.00 -> 8.26 mm, vias 0 -> 1
- net RXIP: track 9.26 -> 1.33 mm, vias 1 -> 0
- net nRESET: track 21.2 -> 13.6 mm, vias 2 -> 1
- net Net-(C18-Pad1): track 0.00 -> 7.41 mm, vias 0 -> 1
- net RXIN: track 9.26 -> 2.27 mm, vias 1 -> 0
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- added copper zone on F.Cu, net SHD
Other:
- net class Default removed
- board text added: "Copyright Tinkerforge GmbH 2020. This documentation describes Open Hardware and is licensed under the CERN OHL v. 1.1. You may redistribute and modify this documentation under the terms of the CERN OHL v.1.1. (http://ohwr.org/cernohl). This documentation is distributed WITHOUT ANY EXPRESS OR IMPLIED WARRANTY, INCLUDING OF MERCHANTABILITY, SATISFACTORY QUALITY AND FITNESS FOR A PARTICULAR PURPOSE.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"
- board text added: "Ethernet Extension w/o PoE 1.1"
- board text removed: "Copyright Tinkerforge GmbH 2015. This documentation describes Open Hardware and is licensed under the CERN OHL v. 1.1. You may redistribute and modify this documentation under the terms of the CERN OHL v.1.1. (http://ohwr.org/cernohl). This documentation is distributed WITHOUT ANY EXPRESS OR IMPLIED WARRANTY, INCLUDING OF MERCHANTABILITY, SATISFACTORY QUALITY AND FITNESS FOR A PARTICULAR PURPOSE.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"
- board text removed: "Ethernet Extension w/o PoE 1.0"
