File: hardware/poe/ethernet-extension-poe.kicad_pcb (KiCad board)
At the start: 4 copper layers, 40 x 40 mm, 121 parts, among them J1 STACK-UP-HIGH, J2 STACK-DOWN, J3 STACK-UP-HIGH, J4 STACK-DOWN, P1 RJPSL-001TA1, P2 CONN_1, Q1 2N7002P, Q2 MMBTA42, Q3 FDC2512, T1 EFD15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

Commit message: version 1.2
Parts:
- removed FILTER1: Filter-8x, DFN16-33x135
- removed P2: CONN_1, con
- added D301: BAS16H, SOD-123, F.Cu at (158.9, 107.8)
- added P301: CONN_1, kicad-libraries:TSTPT, F.Cu at (156.0, 116.7)
- added R101: 1k, kicad-libraries:R0402E, B.Cu at (167.4, 99.7)
- added R102: DNP, kicad-libraries:R0402E, F.Cu at (167.0, 98.5)
- added R301: 510, kicad-libraries:R0805E, F.Cu at (160.7, 110.7)
- added RP101: 82, kicad-libraries:4X0402, B.Cu at (167.4, 97.5)
- C35: footprint C0805 -> kicad-libraries:C0805E
- C39: footprint C0603 -> kicad-libraries:C0805
- D1, D2: footprint kicad-libraries:MiniDIP -> MiniDIP
- G***: moved to B.Cu
- R18, R21: footprint R0603 -> kicad-libraries:R0402F
- R22: footprint R0603 -> kicad-libraries:R0805E
- R24: footprint R0603 -> kicad-libraries:R0805
- T1: footprint kicad-libraries:EFD15 -> EFD15
- moved C33 18.4 mm to (158.5, 120.2), turned to 0 degrees
- moved D5 17.0 mm to (148.4, 114.2)
- moved Q1 14.6 mm to (150.9, 112.9), turned to 270 degrees
- moved D3 14.1 mm to (140.8, 108.8), turned to 90 degrees
- moved R17 13.7 mm to (149.9, 115.6), turned to 270 degrees
- moved R18 13.0 mm to (150.0, 117.5), turned to 180 degrees
- moved Q3 12.5 mm to (156.8, 126.4)
- moved L5 12.3 mm to (154.2, 108.8), turned to 180 degrees
- moved R19 10.5 mm to (154.4, 127.0), turned to 90 degrees
- moved D8 10.5 mm to (152.2, 116.8), turned to 270 degrees
- moved C35 10.2 mm to (160.5, 126.0)
- moved R22 10.1 mm to (160.5, 122.7)
- moved C28 9.28 mm to (143.2, 108.2), turned to 90 degrees
- moved G*** 8.83 mm to (162.8, 113.2), turned to 180 degrees
- moved R23 7.86 mm to (155.0, 123.0), turned to 180 degrees
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Connections:
- net Net-(C26-Pad1) renamed SHD
- C35 pad 1: Net-(C35-Pad1) -> SW
- Q3 pad 1: Net-(C35-Pad1) -> SW
- Q3 pad 2: Net-(C35-Pad1) -> SW
- Q3 pad 5: Net-(C35-Pad1) -> SW
- Q3 pad 6: Net-(C35-Pad1) -> SW
- T1 pad 1: Net-(T1-Pad1) -> SW
- T1 pad 3: Net-(T1-Pad3) -> Net-(C33-Pad2)
- T1 pad 5: Net-(C35-Pad1) -> Net-(R301-Pad1)
- T1 pad 6: Net-(C33-Pad2) -> AGND
- U3 pad 6: Net-(U3-Pad6) -> Net-(C28-Pad1)
- U3 pad 8: Net-(U3-Pad8) -> Net-(C28-Pad1)
- U3 pad 9: Net-(U3-Pad9) -> AGND
- U3 pad EP: Net-(P2-Pad1) -> EP
Routing:
- net AGND: track 152.2 -> 71.2 mm, vias 64 -> 51
- net Net-(C33-Pad2): track 130.6 -> 64.5 mm, vias 15 -> 6
- net Net-(C28-Pad1): track 141.9 -> 91.8 mm, vias 11 -> 18
- net Net-(C35-Pad1): track 45.5 -> 0.00 mm, vias 11 -> 0
- net SW: track 0.00 -> 26.6 mm, vias 0 -> 12
- net Net-(C28-Pad2): track 38.4 -> 64.6 mm, vias 4 -> 9
- net Net-(P2-Pad1): track 19.1 -> 0.00 mm, vias 14 -> 0
- net EP: track 0.00 -> 16.2 mm, vias 0 -> 18
- net Net-(Q3-Pad4): track 20.0 -> 4.96 mm, vias 2 -> 0
- net Net-(R19-Pad2): track 3.71 -> 15.1 mm, vias 0 -> 2
- net VAA: track 36.2 -> 25.5 mm, vias 4 -> 2
- net Net-(R301-Pad1): track 0.00 -> 9.10 mm
- net Net-(D8-Pad1): track 12.0 -> 4.16 mm, vias 2 -> 0
- net SHD: track 7.67 -> 12.9 mm, vias 2 -> 11
- net Net-(R17-Pad2): track 4.41 -> 9.06 mm, vias 0 -> 2
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- added copper zone on F.Cu, net SHD
Other:
- rule via_min_size: 0.70104 -> 0.55
- board text added: "Ethernet Extension 1.2"
- board text removed: "Ethernet Extension 1.1"

Commit message: specify reference
Parts:
- D9: value TLV431 -> ZTLV431AFTA

Commit message: specify stuff
Parts:
- T1: value EFD15 -> EFD15 749119350
- U3: value LTC4267D -> LTC4267CDHC
